File: experiments/Electric/TP-0010U001/CAN_BUS/CAN_BUS.kicad_sch (KiCad schematic)
At the start: 5 parts, among them U1 MCP2515-xSO, U2 TJA1051T, Y1 Crystal

Commit message: backup 2025-09-16
Parts:
- added J1: Conn_01x02, Connector_JST:JST_NV_B02P-NV_1x02_P5.00mm_Vertical, symbol Connector_Generic:Conn_01x02
- added R1: R, Resistor_THT:R_Axial_DIN0204_L3.6mm_D1.6mm_P5.08mm_Horizontal, symbol Device:R
Connections:
- net GND: now reaches C2.1
- net GND: now also C1.2, U2.2 (GND)
- net at U1.1 (TXCAN): now also U2.4 (RXD)
- net Interruption: now reaches U1.12 (~{INT})
- net CLOCK: now reaches U1.13 (SCK)
- net MOSI: now reaches U1.14 (SI)
- net MISO: now reaches U1.15 (SO)
- net Chip Select: now reaches U1.16 (~{CS})
- net at U1.17 (~{RESET}): now also R1.1
- net at U1.2 (RXCAN): now also U2.1 (TXD)
- net VCC: now reaches U2.3 (VCC)
- net VCC: now also R1.2
- net at U2.6 (CANL): now also J1.2 (Pin_2)
- net at U2.7 (CANH): now also J1.1 (Pin_1)
Other:
- note added: "LEYENDA"
- moved on the sheet: U2
